File: SimpleEVSE_AVR.kicad_pcb (KiCad board)
At the start: 2 copper layers, 33 x 14 mm, 21 parts, among them J1 Conn_01x05, J4 AVR-ISP-6, Q1 nch, Q2 nch, U1 AP1117-50, U2 ATtiny13A-SU, U3 A1101ELHL

Commit message: - updated to KiCAD v6.0
Other:
- net class Default removed

Commit message: - updated to KiCAD9 - changed LDO from MEA to EMA
Parts:
- U1: value AP1117-50 -> 5V
Connections:
- U1 pad 1: GND -> +12V
- U1 pad 2: +5V -> GND
- U1 pad 3: +12V -> +5V
Routing:
- net +12V: track 21.0 -> 16.3 mm
- net +5V: track 41.6 -> 41.5 mm, vias 5 -> 3
- net GND: vias 9 -> 8
