File: SimpleEVSE_AVR.kicad_sch (KiCad schematic)
At the start: 21 parts

Commit message: - update to KiCAD 8
Parts:
- C1, C2, C3, C4, C6: value (none) -> 100n; footprint (none) -> Capacitor_SMD:C_0805_2012Metric
- C5: value (none) -> 10n; footprint (none) -> Capacitor_SMD:C_0805_2012Metric
- D1, D2: value (none) -> 1N4148; footprint (none) -> Diode_SMD:D_SOD-123
- D3: value (none) -> LED; footprint (none) -> LED_SMD:LED_0805_2012Metric
- J1: value (none) -> Conn_01x05; footprint (none) -> Connector_PinHeader_2.54mm:PinHeader_1x05_P2.54mm_Horizontal
- J4: value (none) -> AVR-ISP-6; footprint (none) -> Connector_PinHeader_2.54mm:PinHeader_2x03_P2.54mm_Vertical
- Q1, Q2: value (none) -> nch; footprint (none) -> Package_TO_SOT_SMD:SOT-23
- R1: value (none) -> 15k; footprint (none) -> Resistor_SMD:R_0805_2012Metric
- R2: value (none) -> 5k6; footprint (none) -> Resistor_SMD:R_0805_2012Metric
- R3: value (none) -> 1k; footprint (none) -> Resistor_SMD:R_0805_2012Metric
- R4: value (none) -> 10k; footprint (none) -> Resistor_SMD:R_0805_2012Metric
- R5: value (none) -> 150R; footprint (none) -> Resistor_SMD:R_0805_2012Metric
- U1: value (none) -> AP1117-50; footprint (none) -> Package_TO_SOT_SMD:SOT-223-3_TabPin2
- U2: value (none) -> ATtiny13A-SU; footprint (none) -> Package_SO:SOIJ-8_5.3x5.3mm_P1.27mm
- U3: value (none) -> A1101ELHL; footprint (none) -> Package_TO_SOT_SMD:SOT-23

Commit message: - updated to KiCAD9 - changed LDO from MEA to EMA
Parts:
- U1: value AP1117-50 -> 5V; symbol Regulator_Linear:AP1117-50 -> Regulator_Linear:LT1129-5.0_SOT223
Connections:
- net +12V: now also U1.1 (VI); no longer U1.3 (VI)
- net +5V: now also U1.3 (VO); no longer U1.2 (VO)
- net GND: now also U1.2 (GND); no longer U1.1 (GND)
Changed lines of the file:
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@@
 (kicad_sch
-	(version 20231120)
+	(version 20250114)
 	(generator "eeschema")
-	(generator_version "8.0")
+	(generator_version "9.0")
 	(paper "A4")
 	(junction
@@
 	)
 	(junction
-		(at 124.46 101.6)
-		(diameter 0)
-		(color 0 0 0 0)
-	)
-	(junction
 		(at 66.04 114.3)
 		(diameter 0)
@@
 	(label "RELAIS"
 		(at 146.05 64.77 0)
-		(fields_autoplaced yes)
 		(effects
 			(font
@@
 	(label "RELAIS"
 		(at 78.74 109.22 0)
-		(fields_autoplaced yes)
 		(effects
 			(font
@@
 	(label "PWM"
 		(at 146.05 67.31 0)
-		(fields_autoplaced yes)
 		(effects
 			(font
@@
 	(label "FB"
 		(at 93.98 87.63 0)
-		(fields_autoplaced yes)
 		(effects
 			(font
@@
 	(label "FB"
 		(at 146.05 74.93 0)
-		(fields_autoplaced yes)
 		(effects
 			(font
@@
 	(label "PWM"
 		(at 74.93 87.63 0)
-		(fields_autoplaced yes)
 		(effects
 			(font
@@
 	)
 	(symbol
-		(lib_id "Regulator_Linear:AP1117-50")
+		(lib_id "Regulator_Linear:LT1129-5.0_SOT223")
 		(at 80.01 53.34 0)
 		(unit 1)
@@
 			)
 		)
-		(property "Value" "AP1117-50"
+		(property "Value" "5V"
 			(at 80.01 45.72 0)
 			(effects
@@
 		)
 		(property "Footprint" "Package_TO_SOT_SMD:SOT-223-3_TabPin2"
-			(at 80.01 48.26 0)
+			(at 80.01 47.625 0)
 			(effects
 				(font
 					(size 1.27 1.27)
+					(italic yes)
 				)
 				(hide yes)
 			)
 		)
-		(property "Datasheet" "http://www.diodes.com/datasheets/AP1117.pdf"
-			(at 82.55 59.69 0)
+		(property "Datasheet" "https://www.analog.com/media/en/technical-documentation/data-sheets/112935ff.pdf"
+			(at 80.01 54.61 0)
 			(effects
 				(font
@@
 			)
 		)
-		(property "Description" ""
+		(property "Description" "700mA Micropower Low drop-out regulator, Fixed Output 5.0V, SOT-223"
 			(at 80.01 53.34 0)
 			(effects
@@
 		)
 	)
+	(embedded_fonts no)
 )
